File: hardware_design v2/dev_kit_f103.sch (EAGLE design)
At the start: 55 parts, among them U2 FT232RLSSOP, Y1 32.768kHz

Commit message: Version 2 was started to design
Parts:
- removed J1: (no value), SparkFun-Connectors:CONN_04
- removed J3: (no value), SparkFun-Connectors:CONN_06SILK_FEMALE_PTH
- added F1: (no value), adafruit:PTCFUSE-1812
- added J2: CON-SD-CARD_MICROSD-2908-05, 52101-101-REV-A_v16:CON-SD-CARD_MICROSD-2908-05
- added J4: (no value), SparkFun-Connectors:CONN_08"
- added REG: (no value), jumper:JP1E
- GRN: value GREEN -> (none)
- RL13: value 470 -> 1k5
- YLW: value YELLOW -> (none)
- renumbered JP1 to BOOT, LED1 to GRN, LED13 to USRL, LED5 to YLW, S1 to RSTBT, S2 to USRBT
Connections:
- new net N$2: CM.+, CM2.1, F1.1, IC1.OUT, REG.1, RM1.2
- net 3.3V: now also F1.2, J2G$1.VDD, REG.2; no longer CM.+, CM2.1, IC1.OUT, J1.4, RM1.2
- net CRX3: now also S4.4; no longer S4.1
- net CS2: no longer J3.1
- net CSCL: now also S4.3; no longer S4.6
- net CSDA: now also S4.6; no longer S4.3
- net CTX3: now also S4.1; no longer S4.4
- net GND: now also IC1.TAB, J2G$1.VSS; no longer J1.1
- net LED: now also J4.3; no longer J3.3
- net MISO2: now also J2G$1.DAT0(DO)
- net MOSI2: now also J2G$1.CMD(DI)
- net PA0: now also J4.1
- net PA1: no longer FRST.4
- net PA4: now also ADC.6; no longer FRST.3
- net PA5: now also ADC.5; no longer ADC.3
- net PA7: now also ADC.3; no longer ADC.5
- net PA8: now also J2G$1.CD/DAT3(!CS!)
- net PB0: now also FRST.3; no longer ADC.6
- net PB1: now also FRST.4
- net PB3: now also J4.6; no longer J3.6
- net PB4: now also J4.5; no longer J3.5
- net PB5: now also J4.4; no longer J3.4
- net PB8: now also J4.2; no longer J3.2
- net RX3/SDA2: now also S4.5; no longer S4.2
- net SCK2: now also J2G$1.CLK(SCK)
- net SWCLK: now also J4.7; no longer J1.2
- net SWDIO: now also J4.8; no longer J1.3
- net TX3/SCL2: now also S4.2; no longer S4.5
Other:
- note added: "LED"
- note added: "PA0"
- note added: "PA1"
- note added: "PA11"
- note added: "PA12"
- note added: "PA15"
- note added: "PA4"
- note added: "PA5"
- note added: "PA6"
- note added: "PA7"
- note added: "PA8"
- note added: "PB0"
- note added: "PB1"
- note added: "PB3"
- note added: "PB4"
- note added: "PB5"
- note added: "PB8"
