File: hardware_design v4/dev_kit_f103v4.brd (EAGLE design)
At the start: 60.9 x 67 mm, 57 parts, among them J2 CON-SD-CARD_MICROSD-2908-05, U2 FT232RLSSOP, Y1 32.768kHz

Commit message: Hardware design v4 was completed, it is waiting for checking
Parts:
- moved J1 5.08 mm to (62.2, 29.5)
- moved FRST 5.08 mm to (62.2, 7.62)
- moved ADC 3.81 mm to (14.0, 7.62)
- moved PWR 3.81 mm to (14.0, 25.4)
- moved C6 0.24 mm to (51.3, 9.07)
- moved C7 0.24 mm to (48.7, 6.76)
- moved JP3 0.24 mm to (55.5, 4.09)
- moved RD1 0.24 mm to (47.4, 4.45)
- moved RL 0.24 mm to (48.2, 9.14)
- moved C3 0.13 mm to (26.4, 27.2)
Connections:
- net CS2: now also J1.3; no longer J1.8
- net PA15: now also J1.8; no longer J1.1
- net RX2: now also J1.1; no longer J1.2
- net TX2: now also J1.2; no longer J1.3
Routing:
- net 3.3V: track 52.8 -> 319.9 mm, vias 0 -> 8
- net BUTTON: track 2.11 -> 66.6 mm
- net SCL1: track 0.00 -> 52.7 mm, vias 0 -> 1
- net MISO2: track 10.0 -> 61.5 mm
- net SDA1: track 0.00 -> 45.0 mm, vias 0 -> 1
- net SCK2: track 17.0 -> 61.5 mm
- net MOSI2: track 17.9 -> 57.0 mm
- net TX2: track 0.00 -> 34.7 mm, vias 0 -> 1
- net RX2: track 0.00 -> 32.8 mm, vias 0 -> 1
- net PA15: track 0.00 -> 29.7 mm, vias 0 -> 1
- net CTX3: track 0.00 -> 29.2 mm
- net TX3/SCL2: track 0.00 -> 25.6 mm, vias 0 -> 2
- net PA8: track 35.2 -> 60.3 mm, vias 2 -> 4
- net CSCL: track 0.00 -> 24.8 mm
- net RX3/SDA2: track 0.00 -> 22.3 mm, vias 0 -> 2
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Other:
- board size 60.9 x 67 mm -> 56.8 x 69.3 mm
