File: hardware_design v4/dev_kit_f103v4.sch (EAGLE design)
At the start: 50 parts, among them U2 FT232RLSSOP, U7 AMS1117-3.3, Y1 32.768kHz

Commit message: Hardware design v4 was completed, it is waiting for checking
Parts:
- removed F: 0.75A, SparkFun-Fuses:PPTC_THREE-QUARTER-AMP
- removed JP1: (no value), jumper:JP1E
- removed LED1: GREEN, adafruit:LEDCHIP-LED0603
- removed LED4: (no value), adafruit:LEDCHIP-LED0603
- removed LED5: YELLOW, adafruit:LEDCHIP-LED0603
- removed RC1, RC4: 22uF, SparkFun-Capacitors:10UF-POLAR-EIA3528-20V-10%(TANT)
- removed RC2, RC3: 100nF, SparkFun-Capacitors:0.1UF-0603-25V-(+80/-20%)
- removed RD: Red, SparkFun-LED:LED-RED0603-SMART
- removed RGD: 1A/23V, SparkFun-DiscreteSemi:DIODE-SCHOTTKY-BAT20J
- removed RRO: 1.5k, SparkFun-Resistors:2.0KOHM1/10W5%(0603)
- removed RRO3: 470, SparkFun-Resistors:2.0KOHM1/10W5%(0603)
- removed RRO4: 10k, SparkFun-Resistors:2.0KOHM1/10W5%(0603)
- removed RRO5: 330, SparkFun-Resistors:2.0KOHM1/10W5%(0603)
- removed S1, S2: MOMENTARY-SWITCH-SPST-SMD-6.0X3.5MM, SparkFun-Switches:MOMENTARY-SWITCH-SPST-SMD-6.0X3.5MM
- removed SCND: (no value), SparkFun-Connectors:CONN_10"
- removed U7: AMS1117-3.3, AMS1117-3.3:AMS1117-3.3
- added BOOT, REG: (no value), jumper:JP1E
- added CM, CM1: 10uF, SparkFun-Capacitors:10UF-POLAR-EIA3528-20V-10%(TANT)
- added CM2: 100nF, SparkFun-Capacitors:0.1UF-0603-25V-(+80/-20%)
- added D1, D2: (no value), 1N4007:3ASCHOOTKY
- added F1: (no value), adafruit:PTCFUSE-1812
- added FLASH: (no value), W25Q64:W25Q64
- added GRN, USRL, YLW: (no value), adafruit:LEDCHIP-LED0603
- added IC1: (no value), MIC29302WU:MIC29302WU
- added J1: (no value), SparkFun-Connectors:CONN_13
- added J2: CON-SD-CARD_MICROSD-2908-05, 52101-101-REV-A_v16:CON-SD-CARD_MICROSD-2908-05
- added J4: (no value), SparkFun-Connectors:CONN_08"
- added RBOT1: 330, SparkFun-Resistors:2.0KOHM1/10W5%(0603)
- added RBOT2: 10k, SparkFun-Resistors:2.0KOHM1/10W5%(0603)
- added RD1: Red, SparkFun-LED:LED-RED0603-SMART
- added RL: 1.5k, SparkFun-Resistors:2.0KOHM1/10W5%(0603)
- added RL13: 1k5, SparkFun-Resistors:2.0KOHM1/10W5%(0603)
- added RM1: 316, SparkFun-Resistors:2.0KOHM1/10W5%(0603)
- added RM2: 187, SparkFun-Resistors:2.0KOHM1/10W5%(0603)
- added RSTBT, USRBT: MOMENTARY-SWITCH-SPST-SMD-6.0X3.5MM, SparkFun-Switches:MOMENTARY-SWITCH-SPST-SMD-6.0X3.5MM
- added S4: (no value), step_switch:452403012014
- R1, R2: value 470 -> 1k
Connections:
- removed net MISO1: U1A.PA6
- removed net MOSI1: U1A.PA7
- removed net N$10: U1A.PB1
- removed net N$11: U1A.PB12
- removed net N$12: U1A.PB13
- removed net N$13: U1A.PB14
- removed net N$14: U1A.PB15
- removed net N$15: U1A.PB3
- removed net N$16: U1A.PB4
- removed net N$17: U1A.PB5
- removed net N$18: U1A.PB8
- removed net N$19: U1A.PB9
- removed net N$21: U1A.PA1
- removed net N$22: U1A.PA4
- removed net N$23: U1A.PA8
- removed net N$24: U1A.PA11
- removed net N$25: U1A.PA12
- removed net N$26: U1A.PA13
- removed net N$27: U1A.PA14
- removed net N$28: U1A.PA15
- removed net N$29: FRST.8
- removed net N$30: FRST.7
- removed net N$31: FRST.6
- removed net N$32: FRST.5
- removed net N$33: FRST.4
- removed net N$34: FRST.3
- removed net N$9: U1A.PB0
- removed net SCK1: U1A.PA5
- new net CRX3: J1.11, S4.1
- new net CS2: FLASH.CS, J1.3, U1A.PB12
- new net CSCL: J1.10, S4.6
- new net CSDA: J1.9, S4.3
- new net CTX3: J1.12, S4.4
- new net MISO2: FLASH.DO, J1.5, J2G$1.DAT0(DO), U1A.PB14
- new net MOSI2: FLASH.DI, J1.4, J2G$1.CMD(DI), U1A.PB15
- new net N$35: RD1.C, RL.1
- new net PA11: FRST.7, U1A.PA11
- new net PA12: FRST.8, U1A.PA12
- new net PA15: J1.8, U1A.PA15
- new net PA4: ADC.6, U1A.PA4
- new net PA5: ADC.5, U1A.PA5
- new net PA6: ADC.4, U1A.PA6
- new net PA7: ADC.3, U1A.PA7
- new net PA8: FRST.6, J2G$1.CD/DAT3(!CS!), U1A.PA8
- new net PB3: J4.6, U1A.PB3
- new net PB4: J4.5, U1A.PB4
- new net PB5: J4.4, U1A.PB5
- new net PB8: J4.2, U1A.PB8
- new net SCK2: FLASH.CLK, J1.6, J2G$1.CLK(SCK), U1A.PB13
- new net SWCLK: J4.7, U1A.PA14
- new net SWDIO: J4.8, U1A.PA13
- net 3.3V: now also BOOT.2, F1.2, FLASH.H/R, FLASH.VCC, FLASH.WP, J2G$1.VDD, PWR.5, RD1.A, REG.2, USRBT.2; no longer F.2, JP1.2, RD.A, S2.2
- net BUTTON: now also J1.13, RBOT1.2, RBOT2.1, U1A.PB9; no longer RRO4.1, RRO5.2
- net GND: now also CM.-, CM1.-, CM2.2, FLASH.GND, IC1.GND, IC1.TAB, J1.7, J2G$1.VSS, PWR.2, PWR.3, RBOT2.2, RL.2, RL13.2, RM2.2, RSTBT.1; no longer RC1.-, RC2.2, RC3.2, RC4.-, RRO.2, RRO3.2, RRO4.2, S1.1, U7.ADJ/GND
- net LED: now also J4.3, USRL.A; no longer LED4.A
- net N$1: now also CM1.+, D1.OUT, D2.OUT, IC1.EN, IC1.VIN; no longer F.1, RC3.1, RC4.+, U7.VOUT
- net N$2: now also CM.+, CM2.1, F1.1, IC1.OUT, REG.1, RM1.2; no longer RD.C, RRO.1
- net N$20: now also IC1.ADJ, RM1.1, RM2.1; no longer U1A.PA0-WKUP
- net N$3: now also BOOT.1; no longer JP1.1
- net N$4: now also RL13.1, USRL.C; no longer LED4.C, RRO3.1
- net N$5: now also RBOT1.1, USRBT.1; no longer RRO5.1, S2.1
- net N$6: now also GRN.A; no longer LED1.A
- net N$7: now also YLW.A; no longer LED5.A
- net NRST: now also PWR.6, RSTBT.2; no longer S1.2
- net PA0: now also J4.1, U1A.PA0-WKUP; no longer ADC.6
- net PA1: now also FRST.5, U1A.PA1; no longer ADC.5
- net PB0: now also FRST.3, U1A.PB0; no longer ADC.4
- net PB1: now also FRST.4, U1A.PB1; no longer ADC.3
- net RX2: now also J1.1
- net RX3/SDA2: now also S4.5
- net RXLED: now also YLW.C; no longer LED5.C
- net TX2: now also J1.2
- net TX3/SCL2: now also S4.2
- net TXLED: now also GRN.C; no longer LED1.C
- net VCC: no longer R1.2, R2.2
- net VIN: now also D2.IN, PWR.1; no longer RC1.+, RC2.1, RGD.C, U7.VIN
- net V_USB: now also D1.IN, PWR.4, PWR.7, R1.2, R2.2; no longer RGD.A
Other:
- note added: "BOOT"
- note added: "CONNECTOR"
- note added: "CRX3, CTX3, CS2, BUTTON"
- note added: "CRYSTAL OSCILLATORS"
- note added: "FLASH"
- note added: "LED"
- note added: "LED, SWITCH AND BUTTON"
- note added: "MCU"
- note added: "MCU POWER"
- note added: "PA0"
- note added: "PA1"
- note added: "PA11"
- note added: "PA12"
- note added: "PA15"
- note added: "PA4"
- note added: "PA5"
- note added: "PA6"
- note added: "PA7"
- note added: "PA8"
- note added: "PB0"
- note added: "PB1"
- note added: "PB3"
- note added: "PB4"
- note added: "PB5"
- note added: "PB8"
- note added: "RESET"
- note added: "SYSTEM POWER"
- note added: "USB PORT"
- moved on the sheet: ADC, C1, C2, C3, C4, C5, C6, C7, C8, C9, FRST, JP2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
